Commit message: Finish E. joints

File: body.urdf (robot description, URDF)
Before this commit: robot robot, 4 links, 3 joints
Links:
- removed link Link0
- removed link Link1
- removed link Link2
- removed link Link3
- added link Backleg, mass 1; collision box size=1 1 1; visual box size=1 1 1
- added link Frontleg, mass 1; collision box size=1 1 1; visual box size=1 1 1
- added link Torso, mass 1; collision box size=1 1 1; visual box size=1 1 1
Joints:
- removed joint Link0_Link1
- removed joint Link1_Link2
- removed joint Link2_Link3
- added joint Torso_Backleg: type revolute, parent Torso, child Backleg, origin xyz=-0.5 0 1 rpy=0 0 0, axis 0 1 0, limit lower=-3.14159 upper=3.14159 effort=0.0 velocity=0.0
- added joint Torso_Frontleg: type revolute, parent Torso, child Frontleg, origin xyz=0.5 0 1 rpy=0 0 0, axis 0 1 0, limit lower=-3.14159 upper=3.14159 effort=0.0 velocity=0.0

Commit message: Add analyze.py

File: body.urdf (robot description, URDF)
Before this commit: robot robot, 3 links, 2 joints
Links:
- removed link Backleg
- removed link Frontleg
- added link BackLeg, mass 1; collision box size=1 1 1; visual box size=1 1 1
- added link FrontLeg, mass 1; collision box size=1 1 1; visual box size=1 1 1
Joints:
- removed joint Torso_Backleg
- removed joint Torso_Frontleg
- added joint Torso_BackLeg: type revolute, parent Torso, child BackLeg, origin xyz=-0.5 0 1 rpy=0 0 0, axis 0 1 0, limit lower=-3.14159 upper=3.14159 effort=0.0 velocity=0.0
- added joint Torso_FrontLeg: type revolute, parent Torso, child FrontLeg, origin xyz=0.5 0 1 rpy=0 0 0, axis 0 1 0, limit lower=-3.14159 upper=3.14159 effort=0.0 velocity=0.0

Commit message: Gave Spot legs

File: body.urdf (robot description, URDF)
Before this commit: robot robot, 9 links, 8 joints
Links:
- removed link BackLeg
- removed link FrontLeg
- removed link LeftLeg
- removed link LowerBackLeg
- removed link LowerFrontLeg
- removed link LowerLeftLeg
- removed link LowerRightLeg
- removed link RightLeg
- added link BackLeftLeg, mass 1; collision box size=0.15 0.1 0.75; visual box size=0.15 0.1 0.75
- added link BackRightLeg, mass 1; collision box size=0.15 0.1 0.75; visual box size=0.15 0.1 0.75
- added link FrontLeftLeg, mass 1; collision box size=0.15 0.1 0.75; visual box size=0.15 0.1 0.75
- added link FrontRightLeg, mass 1; collision box size=0.15 0.1 0.75; visual box size=0.15 0.1 0.75
- added link LowerBackLeftLeg, mass 1; collision box size=0.1 0.1 0.5; visual box size=0.1 0.1 0.5
- added link LowerBackRightLeg, mass 1; collision box size=0.1 0.1 0.5; visual box size=0.1 0.1 0.5
- added link LowerFrontLeftLeg, mass 1; collision box size=0.1 0.1 0.5; visual box size=0.1 0.1 0.5
- added link LowerFrontRightLeg, mass 1; collision box size=0.1 0.1 0.5; visual box size=0.1 0.1 0.5
- link Torso: geometry collision box size=1.5 0.5 0.2; visual box size=1.5 0.5 0.2
Joints:
- removed joint BackLeg_LowerBackLeg
- removed joint FrontLeg_LowerFrontLeg
- removed joint LeftLeg_LowerLeftLeg
- removed joint RightLeg_LowerRightLeg
- removed joint Torso_BackLeg
- removed joint Torso_FrontLeg
- removed joint Torso_LeftLeg
- removed joint Torso_RightLeg
- added joint BackLeftLeg_LowerBackLeftLeg: type revolute, parent BackLeftLeg, child LowerBackLeftLeg, origin xyz=0 0 -0.65 rpy=-0.0 1.5 -0.0, axis 0 1 0, limit lower=-3.14159 upper=3.14159 effort=0.0 velocity=0.0
- added joint BackRightLeg_LowerBackRightLeg: type revolute, parent BackRightLeg, child LowerBackRightLeg, origin xyz=0 0 -0.65 rpy=-0.0 1.5 -0.0, axis 0 1 0, limit lower=-3.14159 upper=3.14159 effort=0.0 velocity=0.0
- added joint FrontLeftLeg_LowerFrontLeftLeg: type revolute, parent FrontLeftLeg, child LowerFrontLeftLeg, origin xyz=0 0 -0.65 rpy=-0.0 1.5 -0.0, axis 0 1 0, limit lower=-3.14159 upper=3.14159 effort=0.0 velocity=0.0
- added joint FrontRightLeg_LowerFrontRightLeg: type revolute, parent FrontRightLeg, child LowerFrontRightLeg, origin xyz=0 0 -0.65 rpy=-0.0 1.5 -0.0, axis 0 1 0, limit lower=-3.14159 upper=3.14159 effort=0.0 velocity=0.0
- added joint Torso_BackLeftLeg: type revolute, parent Torso, child BackLeftLeg, origin xyz=0.675 0.3 2 rpy=0 -0.75 0, axis 0 1 0, limit lower=-3.14159 upper=3.14159 effort=0.0 velocity=0.0
- added joint Torso_BackRightLeg: type revolute, parent Torso, child BackRightLeg, origin xyz=0.675 -0.3 2 rpy=0 -0.75 0, axis 0 1 0, limit lower=-3.14159 upper=3.14159 effort=0.0 velocity=0.0
- added joint Torso_FrontLeftLeg: type revolute, parent Torso, child FrontLeftLeg, origin xyz=-0.675 0.3 2 rpy=0 -0.75 0, axis 0 1 0, limit lower=-3.14159 upper=3.14159 effort=0.0 velocity=0.0
- added joint Torso_FrontRightLeg: type revolute, parent Torso, child FrontRightLeg, origin xyz=-0.675 -0.3 2 rpy=0 -0.75 0, axis 0 1 0, limit lower=-3.14159 upper=3.14159 effort=0.0 velocity=0.0

Commit message: Fix left/right being switched

File: body.urdf (robot description, URDF)
Before this commit: robot robot, 9 links, 8 joints
Links:
- removed link BackRightLeg
- removed link LowerBackRightLeg
- link LowerBackLeftLeg: geometry collision box size=0.1 0.1 0.75; visual box size=0.1 0.1 0.75
- link LowerFrontLeftLeg: geometry collision box size=0.1 0.1 0.75; visual box size=0.1 0.1 0.75
- link LowerFrontRightLeg: geometry collision box size=0.1 0.1 0.75; visual box size=0.1 0.1 0.75
Joints:
- removed joint BackRightLeg_LowerBackRightLeg
- removed joint Torso_BackRightLeg
- joint Torso_BackLeftLeg: origin xyz=0.675 0.3 2 rpy=0 -0.75 0 -> xyz=0.675 -0.3 2 rpy=0 -0.75 0
- joint Torso_FrontLeftLeg: origin xyz=-0.675 0.3 2 rpy=0 -0.75 0 -> xyz=-0.675 -0.3 2 rpy=0 -0.75 0
- joint Torso_FrontRightLeg: origin xyz=-0.675 -0.3 2 rpy=0 -0.75 0 -> xyz=-0.675 0.3 2 rpy=0 -0.75 0

Commit message: Simplify code

File: body.urdf (robot description, URDF)
Before this commit: robot robot, 7 links, 6 joints
Links:
- added link BackRightLeg, mass 1; collision box size=0.15 0.1 0.75; visual box size=0.15 0.1 0.75
- added link LowerBackRightLeg, mass 1; collision box size=0.1 0.1 0.75; visual box size=0.1 0.1 0.75
Joints:
- added joint BackRightLeg_LowerBackRightLeg: type revolute, parent BackRightLeg, child LowerBackRightLeg, origin xyz=0 0 -0.65 rpy=-0.0 1.5 -0.0, axis 0 1 0, limit lower=-3.14159 upper=3.14159 effort=0.0 velocity=0.0
- added joint Torso_BackRightLeg: type revolute, parent Torso, child BackRightLeg, origin xyz=0.675 0.3 2 rpy=0 -0.75 0, axis 0 1 0, limit lower=-3.14159 upper=3.14159 effort=0.0 velocity=0.0

Commit message: Add arm base

File: body.urdf (robot description, URDF)
Before this commit: robot robot, 9 links, 8 joints
Links:
- added link ArmBase, mass 1; collision box size=0.2 0.2 0.2; visual box size=0.2 0.2 0.2
Joints:
- added joint Torso_ArmBase: type revolute, parent Torso, child ArmBase, origin xyz=0.35 1 1.5999999999999999 rpy=0 0 0, axis 0 0 1, limit lower=-3.14159 upper=3.14159 effort=0.0 velocity=0.0
- joint Torso_BackLeftLeg: origin xyz=0.675 -0.3 2 rpy=0 -0.75 0 -> xyz=1.675 0.7 1.4 rpy=0 -0.75 0
- joint Torso_BackRightLeg: origin xyz=0.675 0.3 2 rpy=0 -0.75 0 -> xyz=1.675 1.3 1.4 rpy=0 -0.75 0
- joint Torso_FrontLeftLeg: origin xyz=-0.675 -0.3 2 rpy=0 -0.75 0 -> xyz=0.32499999999999996 0.7 1.4 rpy=0 -0.75 0
- joint Torso_FrontRightLeg: origin xyz=-0.675 0.3 2 rpy=0 -0.75 0 -> xyz=0.32499999999999996 1.3 1.4 rpy=0 -0.75 0

Commit message: Added arm and grabbers

File: body.urdf (robot description, URDF)
Before this commit: robot robot, 10 links, 9 joints
Links:
- added link Arm1, mass 1; collision box size=0.1 0.1 0.65; visual box size=0.1 0.1 0.65
- added link Arm2, mass 1; collision box size=0.1 0.1 0.65; visual box size=0.1 0.1 0.65
- added link Arm3, mass 1; collision box size=0.1 0.1 0.2; visual box size=0.1 0.1 0.2
- added link Grabber1, mass 1; collision box size=0.05 0.05 0.2; visual box size=0.05 0.05 0.2
- added link Grabber2, mass 1; collision box size=0.05 0.05 0.2; visual box size=0.05 0.05 0.2
- added link Wrist, mass 1; collision box size=0.1 0.1 0.05; visual box size=0.1 0.1 0.05
- link ArmBase: geometry collision box size=0.2 0.2 0.1; visual box size=0.2 0.2 0.1
Joints:
- added joint Arm1_Arm2: type revolute, parent Arm1, child Arm2, origin xyz=0 0 0.65 rpy=-0.0 -2.0943951023931953 -0.0, axis 0 1 0, limit lower=-3.14159 upper=3.14159 effort=0.0 velocity=0.0
- added joint Arm2_Arm3: type revolute, parent Arm2, child Arm3, origin xyz=0 0 0.65 rpy=0 -0.5 0, axis 0 1 0, limit lower=-3.14159 upper=3.14159 effort=0.0 velocity=0.0
- added joint Arm3_Wrist: type revolute, parent Arm3, child Wrist, origin xyz=0 0 0.2 rpy=0 0 0.7853981633974483, axis 0 0 1, limit lower=-3.14159 upper=3.14159 effort=0.0 velocity=0.0
- added joint ArmBase_Arm1: type revolute, parent ArmBase, child Arm1, origin xyz=0 0 0.1 rpy=0 1.0471975511965976 0, axis 0 1 0, limit lower=-3.14159 upper=3.14159 effort=0.0 velocity=0.0
- added joint Wrist_Grabber1: type revolute, parent Wrist, child Grabber1, origin xyz=0.05 0 0.05 rpy=0 0 0, axis 0 1 0, limit lower=-3.14159 upper=3.14159 effort=0.0 velocity=0.0
- added joint Wrist_Grabber2: type revolute, parent Wrist, child Grabber2, origin xyz=-0.05 0 0.05 rpy=0 0 0, axis 0 1 0, limit lower=-3.14159 upper=3.14159 effort=0.0 velocity=0.0
- joint Torso_ArmBase: origin xyz=0.35 1 1.5999999999999999 rpy=0 0 0 -> xyz=0.35 1 1.6 rpy=0 0 0
- joint Torso_BackLeftLeg: origin xyz=1.675 0.7 1.4 rpy=0 -0.75 0 -> xyz=1.675 0.7 1.5 rpy=0 -0.75 0
- joint Torso_BackRightLeg: origin xyz=1.675 1.3 1.4 rpy=0 -0.75 0 -> xyz=1.675 1.3 1.5 rpy=0 -0.75 0
- joint Torso_FrontLeftLeg: origin xyz=0.32499999999999996 0.7 1.4 rpy=0 -0.75 0 -> xyz=0.32499999999999996 0.7 1.5 rpy=0 -0.75 0
- joint Torso_FrontRightLeg: origin xyz=0.32499999999999996 1.3 1.4 rpy=0 -0.75 0 -> xyz=0.32499999999999996 1.3 1.5 rpy=0 -0.75 0

Commit message: Improve lower leg joint placement

File: body.urdf (robot description, URDF)
Before this commit: robot robot, 16 links, 15 joints
Joints:
- joint BackLeftLeg_LowerBackLeftLeg: origin xyz=0 0 -0.65 rpy=-0.0 1.5 -0.0 -> xyz=0 -0.05 -0.65 rpy=-0.0 1.5707963267948966 -0.0
- joint BackRightLeg_LowerBackRightLeg: origin xyz=0 0 -0.65 rpy=-0.0 1.5 -0.0 -> xyz=0 0.05 -0.65 rpy=-0.0 1.5707963267948966 -0.0
- joint FrontLeftLeg_LowerFrontLeftLeg: origin xyz=0 0 -0.65 rpy=-0.0 1.5 -0.0 -> xyz=0 -0.05 -0.65 rpy=-0.0 1.5707963267948966 -0.0
- joint FrontRightLeg_LowerFrontRightLeg: origin xyz=0 0 -0.65 rpy=-0.0 1.5 -0.0 -> xyz=0 0.05 -0.65 rpy=-0.0 1.5707963267948966 -0.0
- joint Torso_ArmBase: origin xyz=0.35 1 1.6 rpy=0 0 0 -> xyz=-0.65 0 1.1 rpy=0 0 0
- joint Torso_BackLeftLeg: origin xyz=1.675 0.7 1.5 rpy=0 -0.75 0 -> xyz=0.675 -0.25 1 rpy=0 -0.7853981633974483 0
- joint Torso_BackRightLeg: origin xyz=1.675 1.3 1.5 rpy=0 -0.75 0 -> xyz=0.675 0.25 1 rpy=0 -0.7853981633974483 0
- joint Torso_FrontLeftLeg: origin xyz=0.32499999999999996 0.7 1.5 rpy=0 -0.75 0 -> xyz=-0.675 -0.25 1 rpy=0 -0.7853981633974483 0
- joint Torso_FrontRightLeg: origin xyz=0.32499999999999996 1.3 1.5 rpy=0 -0.75 0 -> xyz=-0.675 0.25 1 rpy=0 -0.7853981633974483 0

Commit message: Fix LOWER_LEG_JOINT sizing

File: body.urdf (robot description, URDF)
Before this commit: robot robot, 16 links, 15 joints
Joints:
- joint BackLeftLeg_LowerBackLeftLeg: origin xyz=0 -0.05 -0.65 rpy=-0.0 1.5707963267948966 -0.0 -> xyz=0 -0.05 -0.675 rpy=-0.0 1.5707963267948966 -0.0
- joint BackRightLeg_LowerBackRightLeg: origin xyz=0 0.05 -0.65 rpy=-0.0 1.5707963267948966 -0.0 -> xyz=0 0.05 -0.675 rpy=-0.0 1.5707963267948966 -0.0
- joint FrontLeftLeg_LowerFrontLeftLeg: origin xyz=0 -0.05 -0.65 rpy=-0.0 1.5707963267948966 -0.0 -> xyz=0 -0.05 -0.675 rpy=-0.0 1.5707963267948966 -0.0
- joint FrontRightLeg_LowerFrontRightLeg: origin xyz=0 0.05 -0.65 rpy=-0.0 1.5707963267948966 -0.0 -> xyz=0 0.05 -0.675 rpy=-0.0 1.5707963267948966 -0.0

Commit message: Update robot body plan & refactor Joint

File: body.urdf (robot description, URDF)
Before this commit: robot robot, 16 links, 15 joints
Links:
- added link BackLeftHip, mass 1; collision box size=0.15 0 0.15; visual box size=0.15 0 0.15
- added link BackRightHip, mass 1; collision box size=0.1 0.1 0.1; visual box size=0.1 0.1 0.1
- added link FrontLeftHip, mass 1; collision box size=0.15 0 0.15; visual box size=0.15 0 0.15
- added link FrontRightHip, mass 1; collision box size=0.15 0 0.15; visual box size=0.15 0 0.15
Joints:
- removed joint Torso_BackLeftLeg
- removed joint Torso_BackRightLeg
- removed joint Torso_FrontLeftLeg
- removed joint Torso_FrontRightLeg
- added joint BackLeftHip_BackLeftLeg: type revolute, parent BackLeftHip, child BackLeftLeg, origin xyz=0 0 0 rpy=0 -0.8726646259971648 0, axis 0 1 0, limit lower=-1.5882496193148399 upper=1.5882496193148399 effort=0.0 velocity=0.0
- added joint BackRightHip_BackRightLeg: type revolute, parent BackRightHip, child BackRightLeg, origin xyz=0 0 0 rpy=0 -0.8726646259971648 0, axis 0 1 0, limit lower=-1.5882496193148399 upper=1.5882496193148399 effort=0.0 velocity=0.0
- added joint FrontLeftHip_FrontLeftLeg: type revolute, parent FrontLeftHip, child FrontLeftLeg, origin xyz=0 0 0 rpy=0 -0.8726646259971648 0, axis 0 1 0, limit lower=-1.5882496193148399 upper=1.5882496193148399 effort=0.0 velocity=0.0
- added joint FrontRightHip_FrontRightLeg: type revolute, parent FrontRightHip, child FrontRightLeg, origin xyz=0 0 0 rpy=0 -0.8726646259971648 0, axis 0 1 0, limit lower=-1.5882496193148399 upper=1.5882496193148399 effort=0.0 velocity=0.0
- added joint Torso_BackLeftHip: type revolute, parent Torso, child BackLeftHip, origin xyz=0.675 -0.25 1 rpy=0 0 0, axis 1 0 0, limit lower=-0.2617993877991494 upper=0.2617993877991494 effort=0.0 velocity=0.0
- added joint Torso_BackRightHip: type revolute, parent Torso, child BackRightHip, origin xyz=0.675 0.25 1 rpy=0 0 0, axis 1 0 0, limit lower=-0.2617993877991494 upper=0.2617993877991494 effort=0.0 velocity=0.0
- added joint Torso_FrontLeftHip: type revolute, parent Torso, child FrontLeftHip, origin xyz=-0.675 -0.25 1 rpy=0 0 0, axis 1 0 0, limit lower=-0.2617993877991494 upper=0.2617993877991494 effort=0.0 velocity=0.0
- added joint Torso_FrontRightHip: type revolute, parent Torso, child FrontRightHip, origin xyz=-0.675 0.25 1 rpy=0 0 0, axis 1 0 0, limit lower=-0.2617993877991494 upper=0.2617993877991494 effort=0.0 velocity=0.0
- joint Arm1_Arm2: limit lower=-3.14159 upper=3.14159 effort=0.0 velocity=0.0 -> lower=-3.141592653589793 upper=3.141592653589793 effort=0.0 velocity=0.0
- joint Arm2_Arm3: limit lower=-3.14159 upper=3.14159 effort=0.0 velocity=0.0 -> lower=-3.141592653589793 upper=3.141592653589793 effort=0.0 velocity=0.0
- joint Arm3_Wrist: limit lower=-3.14159 upper=3.14159 effort=0.0 velocity=0.0 -> lower=-3.141592653589793 upper=3.141592653589793 effort=0.0 velocity=0.0
- joint ArmBase_Arm1: limit lower=-3.14159 upper=3.14159 effort=0.0 velocity=0.0 -> lower=-3.141592653589793 upper=3.141592653589793 effort=0.0 velocity=0.0
- joint BackLeftLeg_LowerBackLeftLeg: limit lower=-3.14159 upper=3.14159 effort=0.0 velocity=0.0 -> lower=-0.6283185307179586 upper=1.9198621771937625 effort=0.0 velocity=0.0; origin xyz=0 -0.05 -0.675 rpy=-0.0 1.5707963267948966 -0.0 -> xyz=0 -0.05 -0.675 rpy=-0.0 1.7453292519943295 -0.0
- joint BackRightLeg_LowerBackRightLeg: limit lower=-3.14159 upper=3.14159 effort=0.0 velocity=0.0 -> lower=-0.6283185307179586 upper=1.9198621771937625 effort=0.0 velocity=0.0; origin xyz=0 0.05 -0.675 rpy=-0.0 1.5707963267948966 -0.0 -> xyz=0 0.05 -0.675 rpy=-0.0 1.7453292519943295 -0.0
- joint FrontLeftLeg_LowerFrontLeftLeg: limit lower=-3.14159 upper=3.14159 effort=0.0 velocity=0.0 -> lower=-0.6283185307179586 upper=1.9198621771937625 effort=0.0 velocity=0.0; origin xyz=0 -0.05 -0.675 rpy=-0.0 1.5707963267948966 -0.0 -> xyz=0 -0.05 -0.675 rpy=-0.0 1.7453292519943295 -0.0
- joint FrontRightLeg_LowerFrontRightLeg: limit lower=-3.14159 upper=3.14159 effort=0.0 velocity=0.0 -> lower=-0.6283185307179586 upper=1.9198621771937625 effort=0.0 velocity=0.0; origin xyz=0 0.05 -0.675 rpy=-0.0 1.5707963267948966 -0.0 -> xyz=0 0.05 -0.675 rpy=-0.0 1.7453292519943295 -0.0
- joint Torso_ArmBase: limit lower=-3.14159 upper=3.14159 effort=0.0 velocity=0.0 -> lower=-3.141592653589793 upper=3.141592653589793 effort=0.0 velocity=0.0
- joint Wrist_Grabber1: limit lower=-3.14159 upper=3.14159 effort=0.0 velocity=0.0 -> lower=-3.141592653589793 upper=3.141592653589793 effort=0.0 velocity=0.0
- joint Wrist_Grabber2: limit lower=-3.14159 upper=3.14159 effort=0.0 velocity=0.0 -> lower=-3.141592653589793 upper=3.141592653589793 effort=0.0 velocity=0.0

Commit message: Update robot to make it grab cube

File: body.urdf (robot description, URDF)
Before this commit: robot robot, 20 links, 19 joints
Joints:
- joint Arm1_Arm2: limit lower=-3.141592653589793 upper=3.141592653589793 effort=0.0 velocity=0.0 -> lower=-0.7853981633974483 upper=0.7853981633974483 effort=0.0 velocity=0.0
- joint Arm2_Arm3: limit lower=-3.141592653589793 upper=3.141592653589793 effort=0.0 velocity=0.0 -> lower=-0.7853981633974483 upper=0.7853981633974483 effort=0.0 velocity=0.0
- joint ArmBase_Arm1: limit lower=-3.141592653589793 upper=3.141592653589793 effort=0.0 velocity=0.0 -> lower=-1.5707963267948966 upper=0.08726646259971647 effort=0.0 velocity=0.0
- joint Torso_ArmBase: limit lower=-3.141592653589793 upper=3.141592653589793 effort=0.0 velocity=0.0 -> lower=-0.17453292519943295 upper=0.17453292519943295 effort=0.0 velocity=0.0
- joint Wrist_Grabber1: limit lower=-3.141592653589793 upper=3.141592653589793 effort=0.0 velocity=0.0 -> lower=-1.5707963267948966 upper=1.5707963267948966 effort=0.0 velocity=0.0
- joint Wrist_Grabber2: limit lower=-3.141592653589793 upper=3.141592653589793 effort=0.0 velocity=0.0 -> lower=-1.5707963267948966 upper=1.5707963267948966 effort=0.0 velocity=0.0

Commit message: Update robot and brain for A/B testing

File: body.urdf (robot description, URDF)
Before this commit: robot robot, 20 links, 19 joints
Joints:
- joint Torso_BackLeftHip: limit lower=-0.2617993877991494 upper=0.2617993877991494 effort=0.0 velocity=0.0 -> lower=-0.0 upper=0.0 effort=0.0 velocity=0.0
- joint Torso_BackRightHip: limit lower=-0.2617993877991494 upper=0.2617993877991494 effort=0.0 velocity=0.0 -> lower=-0.0 upper=0.0 effort=0.0 velocity=0.0
- joint Torso_FrontLeftHip: limit lower=-0.2617993877991494 upper=0.2617993877991494 effort=0.0 velocity=0.0 -> lower=-0.0 upper=0.0 effort=0.0 velocity=0.0
- joint Torso_FrontRightHip: limit lower=-0.2617993877991494 upper=0.2617993877991494 effort=0.0 velocity=0.0 -> lower=-0.0 upper=0.0 effort=0.0 velocity=0.0
